Commit message: New arduino packages

File: deliverybot_description/urdf/deliverybot.urdf (robot description, URDF)
Before this commit: robot deliverybot, 3 links, 2 joints
Links:
- link base_link: geometry visual mesh filename=file://home/home/liamd/catkin_ws/src/delivery_bot/deliveryb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 scale=0.0010 0.0010 0.0010
