Commit message: Full Ackermann Drive system

File: deliverybot_description/urdf/eva_mesh.urdf (robot description, URDF)
Before this commit: robot eva, 6 links, 5 joints
Links:
- added link chasis_link, mass 64.3; collision mesh filename=package://deliverybot_description/models/EVA_Body.dae; visual mesh filename=package://deliverybot_description/models/EVA_Body.dae
- added link left_wheel_assembly, mass 0.2; collision cylinder length=0.01 radius=0.005; visual cylinder length=0.01 radius=0.005
- added link right_wheel_assembly, mass 0.2; collision cylinder length=0.01 radius=0.005; visual cylinder length=0.01 radius=0.005
- link base_link: geometry 
- link bl_tire: mass None -> 3.512; geometry collision mesh filename=package://deliverybot_description/models/EVA_Wheel.dae; visual mesh filename=package://deliverybot_description/models/EVA_Wheel.dae
- link br_tire: mass None -> 3.512; geometry collision mesh filename=package://deliverybot_description/models/EVA_Wheel.dae; visual mesh filename=package://deliverybot_description/models/EVA_Wheel.dae
- link door: mass None -> 8; geometry collision mesh filename=package://deliverybot_description/models/EVA_Lid.dae; visual mesh filename=package://deliverybot_description/models/EVA_Lid.dae
- link fl_tire: mass None -> 3.512; geometry collision mesh filename=package://deliverybot_description/models/EVA_Wheel.dae; visual mesh filename=package://deliverybot_description/models/EVA_Wheel.dae
- link fr_tire: mass None -> 3.512; geometry collision mesh filename=package://deliverybot_description/models/EVA_Wheel.dae; visual mesh filename=package://deliverybot_description/models/EVA_Wheel.dae
Joints:
- added joint dummy_joint: type fixed, parent base_link, child chasis_link
- added joint left_wheel_hinge: type revolute, parent chasis_link, child left_wheel_assembly, origin xyz=-0.270 0.3 0 rpy=0 0 0, axis 0 0 1, limit lower=-0.75 upper=0.75 effort=100 velocity=1
- added joint right_wheel_hinge: type revolute, parent chasis_link, child right_wheel_assembly, origin xyz=0.270 0.3 0 rpy=0 0 0, axis 0 0 1, limit lower=-0.75 upper=0.75 effort=100 velocity=1
- joint bl_tire_joint: origin xyz=-0.25 -0.3 0.125 rpy=0 0 0 -> xyz=-0.270 -0.3 0 rpy=0 0 0; parent base_link -> chasis_link
- joint br_tire_joint: origin xyz=0.25 -0.3 0.125 rpy=0 0 3.14 -> xyz=0.270 -0.3 0 rpy=0 0 3.14; parent base_link -> chasis_link
- joint door_link: limit lower=0 upper=1.57 effort=0 velocity=0.785 -> lower=0 upper=1.57 effort=100 velocity=0.500; origin xyz=0 -0.4375 .825 rpy=0 0 0 -> xyz=0 -0.4375 .725 rpy=0 0 0; parent base_link -> chasis_link
- joint fl_tire_joint: axis (none) -> 1 0 0; limit (none) -> effort=100 velocity=50; origin xyz=-0.25 0.3 0.125 rpy=0 0 0 -> xyz=0 0 0 rpy=0 0 0; parent base_link -> left_wheel_assembly
- joint fr_tire_joint: axis (none) -> 1 0 0; limit (none) -> effort=100 velocity=50; origin xyz=0.25 0.3 0.125 rpy=0 0 3.14 -> xyz=0 0 0 rpy=0 0 3.14; parent base_link -> right_wheel_assembly
