Commit message: With simulation

File: deliverybot_description/urdf/steer_bot.urdf.xacro (robot description, xacro)
@@ -47,6 +47,8 @@
   <xacro:property name="steer_offset" value="-0.15" />
   <!-- Base link -->
+  <!--
     <link name="dummy">
     </link>
+  -->
     <link name="base_link">
       <visual>
@@ -68,8 +70,10 @@
       </inertial>
     </link>
+<!--
     <joint name="dummy_joint" type="fixed">
       <parent link="dummy" />
       <child link="base_link"/>
     </joint>
+-->
   <!-- Front steer and rear wheel joints required for ackermann_steering_controller -->
     <xacro:front_steer
@@ -148,4 +152,9 @@
   <!-- Colour -->
   <!-- Door Joint -->
+  <xacro:door
+    name="door"
+    parent="base">
+  </xacro:door>
+<!--
     <link name="door">
       <inertial>
@@ -183,3 +192,4 @@
       </joint>
     </transmission>
+-->
 </robot>

File: deliverybot_description/urdf/wheel.xacro (robot description, xacro)
@@ -110,5 +110,5 @@
       </visual>
       <collision>
-        <origin xyz="0 0 0" rpy="0 1.57 0"/>
+        <origin xyz="0 0 0" rpy="0 ${model_rotate} 1.57"/>
         <geometry>
           <mesh filename="package://deliverybot_description/models/EVA_Wheel.dae"/>
@@ -304,3 +304,43 @@
     </gazebo>
   </xacro:macro>
+  <xacro:macro name="door"
+  params="
+  name
+  parent">
+    <link name="${name}_link">
+      <visual>
+        <geometry>
+          <mesh filename="package://deliverybot_description/models/EVA_Lid.dae" />
+        </geometry>
+        <origin rpy="0 0 -1.57" xyz="0.425 0 0" />
+      </visual>
+      <collision>
+        <origin rpy="0 0 -1.57" xyz="0.425 0 0" />
+        <geometry>
+          <mesh filename="package://deliverybot_description/models/EVA_Lid.dae" />
+        </geometry>
+      </collision>
+      <inertial>
+        <origin rpy="0 0 -1.57" xyz="0 0 0" />
+        <mass value="8" />
+        <inertia ixx="0.4381" ixy="0" ixz="0" iyy="0.1637" iyz="0.005" izz="0.6" />
+      </inertial>
+    </link>
+    <joint name="${name}_joint" type="revolute">
+      <limit lower="0" upper="-1.57" effort="100" velocity="0.500" />
+      <origin rpy="0 0 0" xyz="-0.4375 0 .725" />
+      <parent link="${parent}_link" />
+      <child link="${name}_link" />
+      <axis xyz="0 1 0" rpy="0 0 0" />
+    </joint>
+    <transmission name="${name}_hinge_trans">
+      <type>transmission_interface/SimpleTransmission</type>
+      <actuator name="${name}_motor">
+        <mechanicalReduction>1</mechanicalReduction>
+      </actuator>
+      <joint name="${name}_joint">
+        <hardwareInterface>hardware_interface/EffortJointInterface</hardwareInterface>
+      </joint>
+    </transmission>
+  </xacro:macro>
 </robot>
