Commit message: URDF parsed - Scene added

File: deliverybot_description/robot/deliverybot_wheel.xacro (robot description, xacro)
@@ -253,5 +253,5 @@
         </link>
         <joint name="${name}_joint" type="revolute">
-            <limit lower="0" upper="1.57" effort="100" velocity="0.5" />
+            <limit lower="-1.57" upper="0" effort="100" velocity="0.5" />
             <origin rpy="0 0 0" xyz="-0.4375 0 0.725" />
             <parent link="${parent}_link" />
