Commit message: Fixed xacro tree and added subfolder launch convention

File: deliverybot_description/robot/deliverybot.xacro (robot description, xacro)
@@ -73,8 +73,14 @@
         name="rear"
         parent="base"
-        wheel_radius="${wheel_radius/4}"
-        wheel_thickness="${wheel_thickness/2}"
-        wheel_mass="${wheel_mass/32}">
-        <origin xyz="${-base_length/2+axle_offset} 0 0" rpy="${-90 * deg_to_rad} 0 0" />
+        steer_radius="${steer_radius}"
+        steer_thickness="${steer_thickness}"
+        steer_mass="${steer_mass}"
+        wheel_radius="${wheel_radius}"
+        wheel_thickness="${wheel_thickness}"
+        wheel_mass="${wheel_mass/32}"
+        base_length="${base_length}"
+        base_width="${base_width}"
+        axle_offset="${axle_offset}"
+        steer_height="${wheel_radius+steer_offset}">
     </xacro:rear_wheel>
     <!-- Steerable Front Wheels -->
@@ -118,20 +124,26 @@
         name="rear_right"
         parent="base"
+        reflect="-1"
         wheel_radius="${wheel_radius}"
         wheel_thickness="${wheel_thickness}"
         wheel_mass="${wheel_mass}"
-        model_rotate="-1.57">
-        <origin xyz="${-base_length/2+axle_offset} ${-base_width/2-axle_offset} 0"
-            rpy="${-90*deg_to_rad} 0 0" />
+        model_rotate="-1.57"
+        base_length="${base_length}"
+        base_width="${base_width}"
+        axle_offset="${axle_offset}"
+        steer_height="${wheel_radius+steer_offset}">
     </xacro:rear_wheel_lr>
     <xacro:rear_wheel_lr
         name="rear_left"
         parent="base"
+        reflect="1"
         wheel_radius="${wheel_radius}"
         wheel_thickness="${wheel_thickness}"
         wheel_mass="${wheel_mass}"
-        model_rotate="1.57">
-        <origin xyz="${-base_length/2+axle_offset} ${+base_width/2+axle_offset} 0"
-            rpy="${-90*deg_to_rad} 0 0" />
+        model_rotate="1.57"
+        base_length="${base_length}"
+        base_width="${base_width}"
+        axle_offset="${axle_offset}"
+        steer_height="${wheel_radius+steer_offset}">
     </xacro:rear_wheel_lr>
     <!-- Door -->

File: deliverybot_description/robot/deliverybot_wheel.xacro (robot description, xacro)
@@ -55,19 +55,25 @@
             name
             parent
+            steer_radius
+            steer_thickness
+            steer_mass
             wheel_radius
             wheel_thickness
             wheel_mass
-            *origin">
+            base_length
+            base_width
+            axle_offset
+            steer_height">
         <link name="${name}_wheel_link">
             <visual>
                 <origin xyz="0 0 0" rpy="0 0 0" />
                 <geometry>
-                    <cylinder radius="${wheel_radius}" length="${wheel_thickness}" />
-                </geometry>
-            </visual>
-            <collision>
-                <origin xyz="0 0 0" rpy="0 0 0" />
-                <geometry>
-                    <cylinder radius="${wheel_radius}" length="${wheel_thickness}" />
+                    <cylinder radius="${wheel_radius/4}" length="${wheel_thickness/2}" />
+                </geometry>
+            </visual>
+            <collision>
+                <origin xyz="0 0 0" rpy="0 0 0" />
+                <geometry>
+                    <cylinder radius="${wheel_radius/4}" length="${wheel_thickness/2}" />
                 </geometry>
             </collision>
@@ -86,5 +92,6 @@
             <parent link="${parent}_link" />
             <child link="${name}_wheel_link" />
-            <xacro:insert_block name="origin" />
+            <origin xyz="${-base_length/2+axle_offset} 0 ${steer_height}"
+                rpy="${-90 * deg_to_rad} 0 0" />
             <axis xyz="0 1 0" />
         </joint>
@@ -179,9 +186,13 @@
         name
         parent
+        reflect
         wheel_radius
         wheel_thickness
         wheel_mass
         model_rotate
-        *origin">
+        base_length
+        base_width
+        axle_offset
+        steer_height">
         <link name="${name}_wheel_link">
             <visual>
@@ -206,5 +217,6 @@
             <parent link="${parent}_link" />
             <child link="${name}_wheel_link" />
-            <xacro:insert_block name="origin" />
+            <origin xyz="${-base_length/2+axle_offset} ${reflect*(base_width/2+axle_offset)} ${steer_height}"
+                rpy="${-90 * deg_to_rad} 0 0" />
             <axis xyz="0 0 1" />
         </joint>

Commit message: Fixed joint controller loading - XACRO fixed

File: deliverybot_description/robot/deliverybot.xacro (robot description, xacro)
@@ -13,6 +13,6 @@
     <!-- Math Constants -->
     <xacro:property name="deg_to_rad" value="0.01745329251994329577" />
-    <xacro:property name="steer_limhigh_deg" value="30"/>
-    <xacro:property name="steer_limlow_deg" value="-30"/>
+    <xacro:property name="steer_limhigh_deg" value="30" />
+    <xacro:property name="steer_limlow_deg" value="-30" />
     <!-- Robot Base Dimensions -->
     <xacro:property name="base_length" value="0.85" />
@@ -147,20 +147,24 @@
         steer_height="${wheel_radius+steer_offset}">
     </xacro:rear_wheel_lr>
-    <!-- Door -->
     <xacro:door
         name="door"
         parent="base">
     </xacro:door>
-    <xacro:steering_control
-        name="front_right"
-        steer_limlow="${steer_limlow_deg * deg_to_rad}"
-        steer_limhigh="${steer_limhigh_deg * deg_to_rad}" />
-    <xacro:steering_control
-        name="front_left"
-        steer_limlow="${steer_limlow_deg * deg_to_rad}"
-        steer_limhigh="${steer_limhigh_deg * deg_to_rad}" />
-    <xacro:door_control
-        name="door"
-        door_limlow="${0 * deg_to_rad}"
-        door_limhigh="${90 * deg_to_rad}" />
+    <ros2_control name="GazeboSystem" type="system">
+        <hardware>
+            <plugin>gazebo_ros2_control/GazeboSystem</plugin>
+        </hardware>
+        <xacro:steering_control
+            name="front_right"
+            steer_limlow="${steer_limlow_deg * deg_to_rad}"
+            steer_limhigh="${steer_limhigh_deg * deg_to_rad}" />
+        <xacro:steering_control
+            name="front_left"
+            steer_limlow="${steer_limlow_deg * deg_to_rad}"
+            steer_limhigh="${steer_limhigh_deg * deg_to_rad}" />
+        <xacro:door_control
+            name="door"
+            door_limlow="${0 * deg_to_rad}"
+            door_limhigh="${90 * deg_to_rad}" />
+    </ros2_control>
 </robot>

File: deliverybot_description/robot/deliverybot_control.xacro (robot description, xacro)
@@ -6,18 +6,13 @@
         steer_limlow
         steer_limhigh">
-        <ros2_control name="GazeboSystem" type="system">
-            <hardware>
-                <plugin>gazebo_ros2_control/GazeboSystem</plugin>
-            </hardware>
-            <joint name="${name}_steer_joint">
-                <command_interface name="position">
-                    <param name="min">${steer_limlow}</param>
-                    <param name="max">${steer_limhigh}</param>
-                </command_interface>
-                <state_interface name="position" />
-                <state_interface name="velocity" />
-                <state_interface name="effort" />
-            </joint>
-        </ros2_control>
+        <joint name="${name}_steer_joint">
+            <command_interface name="position">
+                <param name="min">${steer_limlow}</param>
+                <param name="max">${steer_limhigh}</param>
+            </command_interface>
+            <state_interface name="position" />
+            <state_interface name="velocity" />
+                <!-- <state_interface name="effort" /> -->
+        </joint>
     </xacro:macro>
     <xacro:macro name="door_control"
@@ -26,18 +21,12 @@
         door_limlow
         door_limhigh">
-        <ros2_control name="GazeboSystem" type="system">
-            <hardware>
-                <plugin>gazebo_ros2_control/GazeboSystem</plugin>
-            </hardware>
-            <joint name="${name}_joint">
-                <command_interface name="position">
-                    <param name="min">${door_limlow}</param>
-                    <param name="max">${door_limhigh}</param>
-                </command_interface>
-                <state_interface name="position" />
-                <state_interface name="velocity" />
-                <state_interface name="effort" />
-            </joint>
-        </ros2_control>
+        <joint name="${name}_joint">
+            <command_interface name="position">
+                <param name="min">${door_limlow}</param>
+                <param name="max">${door_limhigh}</param>
+            </command_interface>
+            <state_interface name="position" />
+            <state_interface name="velocity" />
+        </joint>
     </xacro:macro>
 </robot>

Commit message: Added CMD_VEL control of ackermann steering

File: deliverybot_description/robot/deliverybot.xacro (robot description, xacro)
@@ -8,5 +8,6 @@
         <plugin name="gazebo_ros2_control" filename="libgazebo_ros2_control.so">
             <robotNamespace>${robot_namespace}</robotNamespace>
-            <parameters>$(find deliverybot_description)/config/steering_controller_position.yaml</parameters>
+            <!-- <parameters>$(find deliverybot_description)/config/steering_controller_position.yaml</parameters> -->
+            <parameters>$(find deliverybot_description)/config/deliverybot_controller.yaml</parameters>
         </plugin>
     </gazebo>
@@ -28,4 +29,7 @@
     <xacro:property name="steer_thickness" value="0.02" />
     <xacro:property name="steer_mass" value="1" />
+    <!-- Velocity and Movement -->
+    <xacro:property name="velocity_limlow" value="-5.0"/>
+    <xacro:property name="velocity_limhigh" value="8.0"/>
     <!-- Axle Positions -->
     <xacro:property name="axle_offset" value="0.125" />
@@ -167,4 +171,12 @@
             door_limlow="${0 * deg_to_rad}"
             door_limhigh="${90 * deg_to_rad}" />
+        <xacro:velocity_control
+            name="rear_left"
+            velocity_limlow="${velocity_limlow}"
+            velocity_limhigh="${velocity_limhigh}"/>
+        <xacro:velocity_control
+            name="rear_right"
+            velocity_limlow="${velocity_limlow}"
+            velocity_limhigh="${velocity_limhigh}"/>
     </ros2_control>
 </robot>

File: deliverybot_description/robot/deliverybot_control.xacro (robot description, xacro)
@@ -30,3 +30,18 @@
         </joint>
     </xacro:macro>
+    <xacro:macro name="velocity_control"
+        params="
+        name
+        velocity_limlow
+        velocity_limhigh">
+        <joint name="${name}_wheel_joint">
+            <command_interface name="velocity">
+                <param name="min">${velocity_limlow}</param>
+                <param name="max">${velocity_limhigh}</param>
+            </command_interface>
+            <state_interface name="position" />
+            <state_interface name="velocity"/>
+            <state_interface name="effoty"/>
+        </joint>
+    </xacro:macro>
 </robot>
