Commit message: SLAM_Costmap generation - fixed odometry

File: deliverybot_description/models/deliverybot/xacro/nav2.xacro (robot description, xacro)
@@ -6,5 +6,5 @@
         filename="$(find deliverybot_description)/models/deliverybot/xacro/sensors.xacro" />
     <!-- Realsense Camera -->
-    <!-- <xacro:realsense_camera
+    <xacro:realsense_camera
         name="front"
         parent="base_link"
@@ -12,5 +12,5 @@
         mirror="-1">
         <origin xyz="0 0.39875 0.25250" rpy="0 0 ${90*deg_to_rad}" />
-    </xacro:realsense_camera> -->
+    </xacro:realsense_camera>
     <!-- <xacro:realsense_camera
         name="rear"
@@ -20,5 +20,5 @@
         <origin xyz="0 -0.39875 0.25250" rpy="0 0 ${-90 * deg_to_rad}" />
     </xacro:realsense_camera> -->
-    <xacro:depth_camera
+    <!-- <xacro:depth_camera
         name="front"
         parent="base_link"
@@ -26,5 +26,5 @@
         mirror="-1">
         <origin xyz="0 0.39875 0.25250" rpy="0 0 ${90*deg_to_rad}" />
-    </xacro:depth_camera>
+    </xacro:depth_camera> -->
     <xacro:lidar
         name="top"

File: deliverybot_description/models/deliverybot/xacro/sensors.xacro (robot description, xacro)
@@ -1,6 +1,5 @@
 <?xml version="1.0"?>
 <robot name="deliverybot" xmlns:xacro="http://wiki.ros.org/xacro">
-    <xacro:macro
-        name="realsense_camera"
+    <xacro:macro name="realsense_camera"
         params="
         name
@@ -117,6 +116,5 @@
         </gazebo>
     </xacro:macro>
-    <xacro:macro
-        name="lidar"
+    <xacro:macro name="lidar"
         params="
         name
@@ -366,6 +364,6 @@
                 <!-- output -->
                 <publish_odom>true</publish_odom>
-                <publish_odom_tf>true</publish_odom_tf>
-                <publish_wheel_tf>true</publish_wheel_tf>
+                <publish_odom_tf>false</publish_odom_tf>
+                <publish_wheel_tf>false</publish_wheel_tf>
                 <publish_distance>true</publish_distance>
                 <odometry_frame>odom</odometry_frame>
