Commit message: Navigation Stack Integrated

File: deliverybot_description/models/deliverybot/xacro/deliverybot_joints.xacro (robot description, xacro)
@@ -170,5 +170,5 @@
             </visual>
             <collision>
-                <origin rpy="0 0 0" xyz="0 0.400 0.01750" />
+                <origin rpy="0 0 0" xyz="-0.002550 0.400 0.01750" />
                 <geometry>
                     <mesh

File: deliverybot_description/models/deliverybot/xacro/nav2.xacro (robot description, xacro)
@@ -13,5 +13,5 @@
         <origin xyz="0 0.39875 0.25250" rpy="0 0 ${90*deg_to_rad}" />
     </xacro:realsense_camera>
-    <!-- <xacro:realsense_camera
+    <xacro:realsense_camera
         name="rear"
         parent="base_link"
@@ -19,5 +19,5 @@
         mirror="1">
         <origin xyz="0 -0.39875 0.25250" rpy="0 0 ${-90 * deg_to_rad}" />
-    </xacro:realsense_camera> -->
+    </xacro:realsense_camera>
     <!-- <xacro:depth_camera
         name="front"
