Commit message: CMD_VEL Control Gazebo - Door Actuation

File: deliverybot_description/models/deliverybot/xacro/deliverybot.xacro (robot description, xacro)
@@ -1,6 +1,6 @@
 <?xml version="1.0"?>
 <robot name="deliverybot" xmlns:xacro="http://wiki.ros.org/xacro">
-    <xacro:include filename="$(find deliverybot_description)/robot/deliverybot_wheel.xacro" />
-    <xacro:include filename="$(find deliverybot_description)/robot/deliverybot_control.xacro" />
+    <xacro:include filename="$(find deliverybot_description)/models/deliverybot/xacro/deliverybot_wheel.xacro" />
+    <xacro:include filename="$(find deliverybot_description)/models/deliverybot/xacro/deliverybot_control.xacro" />
     <xacro:property name="robot_namespace" value="/deliverybot" />
     <!-- Gazebo Plugins -->
@@ -8,6 +8,5 @@
         <plugin name="gazebo_ros2_control" filename="libgazebo_ros2_control.so">
             <robotNamespace>${robot_namespace}</robotNamespace>
-            <!-- <parameters>$(find deliverybot_description)/config/steering_controller_position.yaml</parameters> -->
-            <parameters>$(find deliverybot_description)/config/deliverybot_controller.yaml</parameters>
+            <parameters>$(find deliverybot_description)/models/deliverybot/config/controllers.yaml</parameters>
         </plugin>
     </gazebo>
@@ -36,5 +35,5 @@
     <xacro:property name="steer_offset" value="-0.15" />
     <!-- Dummy Link -->
-    <link name="dummy" />
+    <link name="base_footprint" />
     <!-- Base Link -->
     <link name="base_link">
@@ -42,5 +41,5 @@
             <origin xyz="0 0 0.40" rpy="0 0 -1.57" />
             <geometry>
-                <mesh filename="package://deliverybot_description/meshes/EVA_Body.dae" />
+                <mesh filename="package://deliverybot_description/models/deliverybot/meshes/EVA_Body.dae" />
             </geometry>
         </visual>
@@ -48,5 +47,5 @@
             <origin xyz="0 0 0.40" rpy="0 0 -1.57" />
             <geometry>
-                <mesh filename="package://deliverybot_description/meshes/EVA_Body.dae" />
+                <mesh filename="package://deliverybot_description/models/deliverybot/meshes/EVA_Body.dae" />
             </geometry>
         </collision>
@@ -58,34 +57,9 @@
     </link>
     <!-- Dummy Joint -->
-    <joint name="dummy_joint" type="fixed">
-        <parent link="dummy" />
+    <joint name="base_link_joint" type="fixed">
+        <origin xyz="0 0 0" />
+        <parent link="base_footprint" />
         <child link="base_link" />
     </joint>
-    <!-- Front steer and rear wheel joints required for ackermann_steering_controller -->
-    <xacro:front_steer
-        name="front"
-        parent="base"
-        steer_radius="${steer_radius}"
-        steer_thickness="${steer_thickness}"
-        steer_mass="${steer_mass}"
-        base_length="${base_length}"
-        base_width="${base_width}"
-        axle_offset="${axle_offset}"
-        steer_height="${wheel_radius+steer_offset}">
-    </xacro:front_steer>
-    <xacro:rear_wheel
-        name="rear"
-        parent="base"
-        steer_radius="${steer_radius}"
-        steer_thickness="${steer_thickness}"
-        steer_mass="${steer_mass}"
-        wheel_radius="${wheel_radius}"
-        wheel_thickness="${wheel_thickness}"
-        wheel_mass="${wheel_mass/32}"
-        base_length="${base_length}"
-        base_width="${base_width}"
-        axle_offset="${axle_offset}"
-        steer_height="${wheel_radius+steer_offset}">
-    </xacro:rear_wheel>
     <!-- Steerable Front Wheels -->
     <xacro:front_wheel_lr

File: deliverybot_description/models/deliverybot/xacro/deliverybot_control.xacro (robot description, xacro)
@@ -13,5 +13,5 @@
             <state_interface name="position" />
             <state_interface name="velocity" />
-                <!-- <state_interface name="effort" /> -->
+            <state_interface name="effort"/>
         </joint>
     </xacro:macro>
@@ -40,7 +40,6 @@
                 <param name="max">${velocity_limhigh}</param>
             </command_interface>
-            <state_interface name="position" />
             <state_interface name="velocity"/>
-            <state_interface name="effoty"/>
+            <state_interface name="effort"/>
         </joint>
     </xacro:macro>

File: deliverybot_description/models/deliverybot/xacro/deliverybot_wheel.xacro (robot description, xacro)
@@ -3,99 +3,6 @@
     <xacro:property name="steer_effort" value="10.0" />
     <xacro:property name="steer_velocity"
-        value="5.0" />
+        value="0.5" />
     <xacro:property name="steer_limit_deg" value="35.0" />
-    <!-- Bicycle model front steering link (required for the steer drive controller) -->
-    <xacro:macro name="front_steer"
-        params="
-        name
-        parent
-        steer_radius
-        steer_thickness
-        steer_mass
-        base_length
-        base_width
-        axle_offset
-        steer_height">
-        <link name="${name}_steer_link">
-            <visual>
-                <origin xyz="0 0 0" rpy="0 0 0" />
-                <geometry>
-                    <cylinder radius="${steer_radius}" length="${steer_thickness}" />
-                </geometry>
-            </visual>
-            <collision>
-                <origin xyz="0 0 0" rpy="0 0 0" />
-                <geometry>
-                    <cylinder radius="${steer_radius}" length="${steer_thickness}" />
-                </geometry>
-            </collision>
-            <inertial>
-                <origin rpy="0 0 0" xyz="0 0 0" />
-                <mass value="${steer_mass}" />
-                <inertia
-                    ixx="${steer_mass * (3.0 * steer_radius * steer_radius + steer_thickness * steer_thickness) / 12.0}"
-                    ixy="0.0" ixz="0.0"
-                    iyy="${steer_mass * (3.0 * steer_radius * steer_radius + steer_thickness * steer_thickness) / 12.0}"
-                    iyz="0.0"
-                    izz="${steer_mass * (steer_radius * steer_radius) / 2.0}" />
-            </inertial>
-        </link>
-        <joint name="${name}_steer_joint" type="revolute">
-            <parent link="${parent}_link" />
-            <child link="${name}_steer_link" />
-            <origin xyz="${base_length/2-axle_offset} 0 ${steer_height}" rpy="0 0 0" />
-            <axis xyz="0 0 1" />
-            <limit effort="${steer_effort}"
-                lower="${-180.0 * deg_to_rad}" upper="${180.0 * deg_to_rad}"
-                velocity="${steer_velocity}" />
-        </joint>
-    </xacro:macro>
-    <xacro:macro name="rear_wheel"
-        params="
-            name
-            parent
-            steer_radius
-            steer_thickness
-            steer_mass
-            wheel_radius
-            wheel_thickness
-            wheel_mass
-            base_length
-            base_width
-            axle_offset
-            steer_height">
-        <link name="${name}_wheel_link">
-            <visual>
-                <origin xyz="0 0 0" rpy="0 0 0" />
-                <geometry>
-                    <cylinder radius="${wheel_radius/4}" length="${wheel_thickness/2}" />
-                </geometry>
-            </visual>
-            <collision>
-                <origin xyz="0 0 0" rpy="0 0 0" />
-                <geometry>
-                    <cylinder radius="${wheel_radius/4}" length="${wheel_thickness/2}" />
-                </geometry>
-            </collision>
-            <inertial>
-                <origin rpy="0 0 0" xyz="0 0 0" />
-                <mass value="${steer_mass}" />
-                <inertia
-                    ixx="${steer_mass * (3.0 * steer_radius * steer_radius + steer_thickness * steer_thickness) / 12.0}"
-                    ixy="0.0" ixz="0.0"
-                    iyy="${steer_mass * (3.0 * steer_radius * steer_radius + steer_thickness * steer_thickness) / 12.0}"
-                    iyz="0.0"
-                    izz="${steer_mass * (steer_radius * steer_radius) / 2.0}" />
-            </inertial>
-        </link>
-        <joint name="${name}_wheel_joint" type="continuous">
-            <parent link="${parent}_link" />
-            <child link="${name}_wheel_link" />
-            <origin xyz="${-base_length/2+axle_offset} 0 ${steer_height}"
-                rpy="${-90 * deg_to_rad} 0 0" />
-            <axis xyz="0 1 0" />
-        </joint>
-    </xacro:macro>
-    <!-- Front Steering Links Xacro -->
     <xacro:macro
         name="front_wheel_lr"
@@ -144,5 +51,5 @@
                 <origin xyz="0 0 0" rpy="0 ${model_rotate} 1.57" />
                 <geometry>
-                    <mesh filename="package://deliverybot_description/meshes/EVA_Wheel.dae" />
+                    <mesh filename="package://deliverybot_description/models/deliverybot/meshes/EVA_Wheel.dae" />
                 </geometry>
             </visual>
@@ -150,5 +57,5 @@
                 <origin xyz="0 0 0" rpy="0 ${model_rotate} 1.57" />
                 <geometry>
-                    <mesh filename="package://deliverybot_description/meshes/EVA_Wheel.dae" />
+                    <mesh filename="package://deliverybot_description/models/deliverybot/meshes/EVA_Wheel.dae" />
                 </geometry>
             </collision>
@@ -199,5 +106,5 @@
                 <origin xyz="0 0 0" rpy="0 ${model_rotate} 1.57" />
                 <geometry>
-                    <mesh filename="package://deliverybot_description/meshes/EVA_Wheel.dae" />
+                    <mesh filename="package://deliverybot_description/models/deliverybot/meshes/EVA_Wheel.dae" />
                 </geometry>
             </visual>
@@ -205,5 +112,5 @@
                 <origin xyz="0 0 0" rpy="0 ${model_rotate} 1.57" />
                 <geometry>
-                    <mesh filename="package://deliverybot_description/meshes/EVA_Wheel.dae" />
+                    <mesh filename="package://deliverybot_description/models/deliverybot/meshes/EVA_Wheel.dae" />
                 </geometry>
             </collision>
@@ -236,5 +143,5 @@
             <visual>
                 <geometry>
-                    <mesh filename="package://deliverybot_description/meshes/EVA_Lid.dae" />
+                    <mesh filename="package://deliverybot_description/models/deliverybot/meshes/EVA_Lid.dae" />
                 </geometry>
                 <origin rpy="0 0 -1.57" xyz="0.425 0 0" />
@@ -243,5 +150,5 @@
                 <origin rpy="0 0 -1.57" xyz="0.425 0 0" />
                 <geometry>
-                    <mesh filename="package://deliverybot_description/meshes/EVA_Lid.dae" />
+                    <mesh filename="package://deliverybot_description/models/deliverybot/meshes/EVA_Lid.dae" />
                 </geometry>
             </collision>

Commit message: Working RVIZ Visualization

File: deliverybot_description/models/deliverybot/xacro/deliverybot.xacro (robot description, xacro)
@@ -152,4 +152,12 @@
             velocity_limlow="${velocity_limlow}"
             velocity_limhigh="${velocity_limhigh}"/>
+        <xacro:velocity_control
+            name="front_right"
+            velocity_limlow="${velocity_limlow}"
+            velocity_limhigh="${velocity_limhigh}"/>
+        <xacro:velocity_control
+            name="front_left"
+            velocity_limlow="${velocity_limlow}"
+            velocity_limhigh="${velocity_limhigh}"/>
     </ros2_control>
 </robot>

File: deliverybot_description/models/deliverybot/xacro/deliverybot_control.xacro (robot description, xacro)
@@ -40,4 +40,5 @@
                 <param name="max">${velocity_limhigh}</param>
             </command_interface>
+            <state_interface name="position" />
             <state_interface name="velocity"/>
             <state_interface name="effort"/>

File: deliverybot_description/models/deliverybot/xacro/deliverybot_wheel.xacro (robot description, xacro)
@@ -51,5 +51,6 @@
                 <origin xyz="0 0 0" rpy="0 ${model_rotate} 1.57" />
                 <geometry>
-                    <mesh filename="package://deliverybot_description/models/deliverybot/meshes/EVA_Wheel.dae" />
+                    <mesh
+                        filename="package://deliverybot_description/models/deliverybot/meshes/EVA_Wheel.dae" />
                 </geometry>
             </visual>
@@ -57,5 +58,6 @@
                 <origin xyz="0 0 0" rpy="0 ${model_rotate} 1.57" />
                 <geometry>
-                    <mesh filename="package://deliverybot_description/models/deliverybot/meshes/EVA_Wheel.dae" />
+                    <mesh
+                        filename="package://deliverybot_description/models/deliverybot/meshes/EVA_Wheel.dae" />
                 </geometry>
             </collision>
@@ -86,4 +88,25 @@
             <fdir1 value="0 1 0" />
         </gazebo>
+        <!-- Transmissions -->
+        <!-- <transmission name="${name}_steer_joint_transmission">
+            <type>transmission_interface/SimpleTransmission</type>
+            <joint name="${name}_steer_joint">
+                <hardwareInterface>hardware_interface/PositionJointInterface</hardwareInterface>
+            </joint>
+            <actuator name="${name}_steer_motor">
+                <hardwareInterface>hardware_interface/PositionJointInterface</hardwareInterface>
+                <mechanicalReduction>1</mechanicalReduction>
+            </actuator>
+        </transmission>
+        <transmission name="{name}_wheel_joint_transmission">
+            <type>transmission_interface/SimpleTransmission</type>
+            <joint name="${name}_wheel_joint">
+                <hardwareInterface>hardware_interface/VelocityJointInterface</hardwareInterface>
+            </joint>
+            <actuator name="${name}_wheel_motor">
+                <hardwareInterface>hardware_interface/VelocityJointInterface</hardwareInterface>
+                <mechanicalReduction>1</mechanicalReduction>
+            </actuator>
+        </transmission> -->
     </xacro:macro>
     <!-- Rear Wheel Links -->
@@ -106,5 +129,6 @@
                 <origin xyz="0 0 0" rpy="0 ${model_rotate} 1.57" />
                 <geometry>
-                    <mesh filename="package://deliverybot_description/models/deliverybot/meshes/EVA_Wheel.dae" />
+                    <mesh
+                        filename="package://deliverybot_description/models/deliverybot/meshes/EVA_Wheel.dae" />
                 </geometry>
             </visual>
@@ -112,5 +136,6 @@
                 <origin xyz="0 0 0" rpy="0 ${model_rotate} 1.57" />
                 <geometry>
-                    <mesh filename="package://deliverybot_description/models/deliverybot/meshes/EVA_Wheel.dae" />
+                    <mesh
+                        filename="package://deliverybot_description/models/deliverybot/meshes/EVA_Wheel.dae" />
                 </geometry>
             </collision>
@@ -124,5 +149,6 @@
             <parent link="${parent}_link" />
             <child link="${name}_wheel_link" />
-            <origin xyz="${-base_length/2+axle_offset} ${reflect*(base_width/2+axle_offset)} ${steer_height}"
+            <origin
+                xyz="${-base_length/2+axle_offset} ${reflect*(base_width/2+axle_offset)} ${steer_height}"
                 rpy="${-90 * deg_to_rad} 0 0" />
             <axis xyz="0 0 1" />
@@ -135,4 +161,14 @@
             <fdir1 value="0 1 0" />
         </gazebo>
+        <!-- <transmission name="{name}_wheel_joint_transmission">
+            <type>transmission_interface/SimpleTransmission</type>
+            <joint name="${name}_wheel_joint">
+                <hardwareInterface>hardware_interface/VelocityJointInterface</hardwareInterface>
+            </joint>
+            <actuator name="${name}_wheel_motor">
+                <hardwareInterface>hardware_interface/VelocityJointInterface</hardwareInterface>
+                <mechanicalReduction>1</mechanicalReduction>
+            </actuator>
+        </transmission> -->
     </xacro:macro>
     <xacro:macro name="door"
@@ -143,12 +179,14 @@
             <visual>
                 <geometry>
-                    <mesh filename="package://deliverybot_description/models/deliverybot/meshes/EVA_Lid.dae" />
-                </geometry>
-                <origin rpy="0 0 -1.57" xyz="0.425 0 0" />
+                    <mesh
+                        filename="package://deliverybot_description/models/deliverybot/meshes/EVA_Lid.dae" />
+                </geometry>
+                <origin rpy="0 0 ${-90 * deg_to_rad}" xyz="0.42375 0 0" />
             </visual>
             <collision>
-                <origin rpy="0 0 -1.57" xyz="0.425 0 0" />
-                <geometry>
-                    <mesh filename="package://deliverybot_description/models/deliverybot/meshes/EVA_Lid.dae" />
+                <origin rpy="0 0 ${-90 * deg_to_rad}" xyz="0.42375 0 0" />
+                <geometry>
+                    <mesh
+                        filename="package://deliverybot_description/models/deliverybot/meshes/EVA_Lid.dae" />
                 </geometry>
             </collision>
@@ -161,5 +199,5 @@
         <joint name="${name}_joint" type="revolute">
             <limit lower="-1.57" upper="0" effort="100" velocity="0.5" />
-            <origin rpy="0 0 0" xyz="-0.4375 0 0.725" />
+            <origin rpy="0 0 0" xyz="-0.4370 0.0025 0.725" />
             <parent link="${parent}_link" />
             <child link="${name}_link" />

Commit message: Improved Ackermann Steering - 4w vel control

File: deliverybot_description/models/deliverybot/xacro/deliverybot.xacro (robot description, xacro)
@@ -1,5 +1,5 @@
 <?xml version="1.0"?>
 <robot name="deliverybot" xmlns:xacro="http://wiki.ros.org/xacro">
-    <xacro:include filename="$(find deliverybot_description)/models/deliverybot/xacro/deliverybot_wheel.xacro" />
+    <xacro:include filename="$(find deliverybot_description)/models/deliverybot/xacro/deliverybot_joints.xacro" />
     <xacro:include filename="$(find deliverybot_description)/models/deliverybot/xacro/deliverybot_control.xacro" />
     <xacro:property name="robot_namespace" value="/deliverybot" />

File: deliverybot_description/models/deliverybot/xacro/deliverybot_control.xacro (robot description, xacro)
@@ -1,4 +1,4 @@
 <?xml version="1.0"?>
-<robot name="deliverybot_wheel" xmlns:xacro="http://wiki.ros.org/xacro">
+<robot name="deliverybot" xmlns:xacro="http://wiki.ros.org/xacro">
     <xacro:macro name="steering_control"
         params="
@@ -13,5 +13,4 @@
             <state_interface name="position" />
             <state_interface name="velocity" />
-            <state_interface name="effort"/>
         </joint>
     </xacro:macro>

File: deliverybot_description/models/deliverybot/xacro/deliverybot_joints.xacro (robot description, xacro)
@@ -1,4 +1,4 @@
 <?xml version="1.0"?>
-<robot name="deliverybot_wheel" xmlns:xacro="http://wiki.ros.org/xacro">
+<robot name="deliverybot" xmlns:xacro="http://wiki.ros.org/xacro">
     <xacro:property name="steer_effort" value="10.0" />
     <xacro:property name="steer_velocity"
@@ -61,4 +61,12 @@
                         filename="package://deliverybot_description/models/deliverybot/meshes/EVA_Wheel.dae" />
                 </geometry>
+                <surface>
+                    <friction>
+                        <ode>
+                            <mu>0.7</mu>
+                            <mu2>0.7</mu2>
+                        </ode>
+                    </friction>
+                </surface>
             </collision>
             <inertial>
@@ -88,25 +96,4 @@
             <fdir1 value="0 1 0" />
         </gazebo>
-        <!-- Transmissions -->
-        <!-- <transmission name="${name}_steer_joint_transmission">
-            <type>transmission_interface/SimpleTransmission</type>
-            <joint name="${name}_steer_joint">
-                <hardwareInterface>hardware_interface/PositionJointInterface</hardwareInterface>
-            </joint>
-            <actuator name="${name}_steer_motor">
-                <hardwareInterface>hardware_interface/PositionJointInterface</hardwareInterface>
-                <mechanicalReduction>1</mechanicalReduction>
-            </actuator>
-        </transmission>
-        <transmission name="{name}_wheel_joint_transmission">
-            <type>transmission_interface/SimpleTransmission</type>
-            <joint name="${name}_wheel_joint">
-                <hardwareInterface>hardware_interface/VelocityJointInterface</hardwareInterface>
-            </joint>
-            <actuator name="${name}_wheel_motor">
-                <hardwareInterface>hardware_interface/VelocityJointInterface</hardwareInterface>
-                <mechanicalReduction>1</mechanicalReduction>
-            </actuator>
-        </transmission> -->
     </xacro:macro>
     <!-- Rear Wheel Links -->
@@ -139,4 +126,12 @@
                         filename="package://deliverybot_description/models/deliverybot/meshes/EVA_Wheel.dae" />
                 </geometry>
+                <surface>
+                    <friction>
+                        <ode>
+                            <mu>0.7</mu>
+                            <mu2>0.7</mu2>
+                        </ode>
+                    </friction>
+                </surface>
             </collision>
             <inertial>
@@ -161,14 +156,4 @@
             <fdir1 value="0 1 0" />
         </gazebo>
-        <!-- <transmission name="{name}_wheel_joint_transmission">
-            <type>transmission_interface/SimpleTransmission</type>
-            <joint name="${name}_wheel_joint">
-                <hardwareInterface>hardware_interface/VelocityJointInterface</hardwareInterface>
-            </joint>
-            <actuator name="${name}_wheel_motor">
-                <hardwareInterface>hardware_interface/VelocityJointInterface</hardwareInterface>
-                <mechanicalReduction>1</mechanicalReduction>
-            </actuator>
-        </transmission> -->
     </xacro:macro>
     <xacro:macro name="door"
