Commit message: RGB and Depth Cameras added to RVIZ + Gazebo

File: deliverybot_description/models/deliverybot/xacro/deliverybot.xacro (robot description, xacro)
@@ -1,6 +1,9 @@
 <?xml version="1.0"?>
 <robot name="deliverybot" xmlns:xacro="http://wiki.ros.org/xacro">
-    <xacro:include filename="$(find deliverybot_description)/models/deliverybot/xacro/deliverybot_joints.xacro" />
-    <xacro:include filename="$(find deliverybot_description)/models/deliverybot/xacro/deliverybot_control.xacro" />
+    <xacro:include
+        filename="$(find deliverybot_description)/models/deliverybot/xacro/deliverybot_joints.xacro" />
+    <xacro:include
+        filename="$(find deliverybot_description)/models/deliverybot/xacro/deliverybot_control.xacro" />
+    <xacro:include filename="$(find deliverybot_description)/models/deliverybot/xacro/cameras.xacro" />
     <xacro:property name="robot_namespace" value="/deliverybot" />
     <!-- Gazebo Plugins -->
@@ -29,6 +32,6 @@
     <xacro:property name="steer_mass" value="1" />
     <!-- Velocity and Movement -->
-    <xacro:property name="velocity_limlow" value="-5.0"/>
-    <xacro:property name="velocity_limhigh" value="8.0"/>
+    <xacro:property name="velocity_limlow" value="-5.0" />
+    <xacro:property name="velocity_limhigh" value="8.0" />
     <!-- Axle Positions -->
     <xacro:property name="axle_offset" value="0.125" />
@@ -39,7 +42,8 @@
     <link name="base_link">
         <visual>
-            <origin xyz="0 0 0.40" rpy="0 0 -1.57" />
+            <origin xyz="0 0 0.325" rpy="0 0 -1.57" />
             <geometry>
-                <mesh filename="package://deliverybot_description/models/deliverybot/meshes/EVA_Body.dae" />
+                <mesh
+                    filename="package://deliverybot_description/models/deliverybot/meshes/EVA_Body_new.dae" />
             </geometry>
         </visual>
@@ -47,5 +51,6 @@
             <origin xyz="0 0 0.40" rpy="0 0 -1.57" />
             <geometry>
-                <mesh filename="package://deliverybot_description/models/deliverybot/meshes/EVA_Body.dae" />
+                <mesh
+                    filename="package://deliverybot_description/models/deliverybot/meshes/EVA_Body_new.dae" />
             </geometry>
         </collision>
@@ -97,5 +102,6 @@
         <origin xyz="0 0 0" rpy="${-90 * deg_to_rad} 0 0" />
     </xacro:front_wheel_lr>
-    <!--Rear Wheels -->
+    <!--Rear
+    Wheels -->
     <xacro:rear_wheel_lr
         name="rear_right"
@@ -128,4 +134,33 @@
         parent="base">
     </xacro:door>
+    <!-- RGB and Depth Cameras -->
+    <xacro:rgb_camera
+        name="front"
+        parent="base_link"
+        orientation="${90 * deg_to_rad}"
+        mirror = "1">
+        <origin xyz="0.39875 0 0.575" rpy="0 0 0" />
+    </xacro:rgb_camera>
+    <xacro:rgb_camera
+        name="rear"
+        parent="base_link"
+        orientation="${-90 * deg_to_rad}"
+        mirror = "-1">
+        <origin xyz="-0.39875 0 0.575" rpy="0 0 ${180 * deg_to_rad}" />
+    </xacro:rgb_camera>
+    <xacro:depth_camera
+        name="front"
+        parent="base_link"
+        orientation="0"
+        mirror = "-1">
+        <origin xyz="0.39875 0 0.575" rpy="0 0 0" />
+    </xacro:depth_camera>
+    <xacro:depth_camera
+        name="rear"
+        parent="base_link"
+        orientation="${-90 * deg_to_rad}"
+        mirror = "-1">
+        <origin xyz="-0.39875 0 0.575" rpy="0 0 ${180 * deg_to_rad}" />
+    </xacro:depth_camera>
     <ros2_control name="GazeboSystem" type="system">
         <hardware>
@@ -147,17 +182,17 @@
             name="rear_left"
             velocity_limlow="${velocity_limlow}"
-            velocity_limhigh="${velocity_limhigh}"/>
+            velocity_limhigh="${velocity_limhigh}" />
         <xacro:velocity_control
             name="rear_right"
             velocity_limlow="${velocity_limlow}"
-            velocity_limhigh="${velocity_limhigh}"/>
+            velocity_limhigh="${velocity_limhigh}" />
         <xacro:velocity_control
             name="front_right"
             velocity_limlow="${velocity_limlow}"
-            velocity_limhigh="${velocity_limhigh}"/>
+            velocity_limhigh="${velocity_limhigh}" />
         <xacro:velocity_control
             name="front_left"
             velocity_limlow="${velocity_limlow}"
-            velocity_limhigh="${velocity_limhigh}"/>
+            velocity_limhigh="${velocity_limhigh}" />
     </ros2_control>
 </robot>

File: deliverybot_description/models/deliverybot/xacro/deliverybot_joints.xacro (robot description, xacro)
@@ -167,8 +167,8 @@
                         filename="package://deliverybot_description/models/deliverybot/meshes/EVA_Lid.dae" />
                 </geometry>
-                <origin rpy="0 0 ${-90 * deg_to_rad}" xyz="0.42375 0 0" />
+                <origin rpy="0 0 ${-90 * deg_to_rad}" xyz="0.42300 0 0" />
             </visual>
             <collision>
-                <origin rpy="0 0 ${-90 * deg_to_rad}" xyz="0.42375 0 0" />
+                <origin rpy="0 0 ${-90 * deg_to_rad}" xyz="0.42300 0 0" />
                 <geometry>
                     <mesh
@@ -184,5 +184,5 @@
         <joint name="${name}_joint" type="revolute">
             <limit lower="-1.57" upper="0" effort="100" velocity="0.5" />
-            <origin rpy="0 0 0" xyz="-0.4370 0.0025 0.725" />
+            <origin rpy="0 0 0" xyz="-0.4365 0.0025 0.695" />
             <parent link="${parent}_link" />
             <child link="${name}_link" />

Commit message: Added RTAB_Map Mapping and Visualization

File: deliverybot_description/models/deliverybot/xacro/deliverybot.xacro (robot description, xacro)
@@ -38,5 +38,6 @@
     <xacro:property name="steer_offset" value="-0.15" />
     <!-- Dummy Link -->
-    <link name="base_footprint" />
+    <!-- <link name="base_footprint" /> -->
+    <!-- <link name="map" /> -->
     <!-- Base Link -->
     <link name="base_link">
@@ -62,9 +63,9 @@
     </link>
     <!-- Dummy Joint -->
-    <joint name="base_link_joint" type="fixed">
-        <origin xyz="0 0 0" />
-        <parent link="base_footprint" />
-        <child link="base_link" />
-    </joint>
+    <!-- <joint name="base_link_joint" type="fixed">
+        <origin xyz="0 0 -0.15" />
+        <parent link="base_link" />
+        <child link="map" />
+    </joint> -->
     <!-- Steerable Front Wheels -->
     <xacro:front_wheel_lr

Commit message: Cleaned URDF - Added Base_Footprint

File: deliverybot_description/models/deliverybot/xacro/deliverybot.xacro (robot description, xacro)
@@ -20,6 +20,6 @@
     <!-- Robot Base Dimensions -->
     <xacro:property name="base_length" value="0.85" />
-    <xacro:property name="base_width" value="0.30" />
-    <xacro:property name="base_length" value="0.75" />
+    <xacro:property name="base_width" value="0.35" />
+    <!-- <xacro:property name="base_length" value="0.75" /> -->
     <xacro:property name="base_mass" value="72.3" />
     <!-- Wheel Link Dimensions -->
@@ -35,13 +35,14 @@
     <xacro:property name="velocity_limhigh" value="8.0" />
     <!-- Axle Positions -->
-    <xacro:property name="axle_offset" value="0.125" />
+    <xacro:property name="axle_length_offset" value="0.125" />
+    <xacro:property name="axle_width_offset" value="0.1"/>
     <xacro:property name="steer_offset" value="-0.15" />
     <!-- Dummy Link -->
-    <!-- <link name="base_footprint" /> -->
+    <link name="base_footprint" />
     <!-- <link name="map" /> -->
     <!-- Base Link -->
     <link name="base_link">
         <visual>
-            <origin xyz="0 0 0.325" rpy="0 0 -1.57" />
+            <origin xyz="0 0 0" rpy="0 0 0" />
             <geometry>
                 <mesh
@@ -50,5 +51,5 @@
         </visual>
         <collision>
-            <origin xyz="0 0 0.40" rpy="0 0 -1.57" />
+            <origin xyz="0 0 0" rpy="0 0 0" />
             <geometry>
                 <mesh
@@ -63,9 +64,9 @@
     </link>
     <!-- Dummy Joint -->
-    <!-- <joint name="base_link_joint" type="fixed">
-        <origin xyz="0 0 -0.15" />
-        <parent link="base_link" />
-        <child link="map" />
-    </joint> -->
+    <joint name="base_joint" type="fixed">
+        <origin xyz="0 0 0.470" rpy="0 0 0"/>
+        <parent link="base_footprint" />
+        <child link="base_link" />
+    </joint>
     <!-- Steerable Front Wheels -->
     <xacro:front_wheel_lr
@@ -81,8 +82,8 @@
         base_length="${base_length}"
         base_width="${base_width}"
-        axle_offset="${axle_offset}"
+        axle_length_offset="${axle_length_offset}"
+        axle_width_offset="${axle_width_offset}"
         steer_height="${wheel_radius+steer_offset}"
-        model_rotate="-1.57">
-        <origin xyz="0 0 0" rpy="${-90 * deg_to_rad} 0 0" />
+        model_rotate="${pi}">
     </xacro:front_wheel_lr>
     <xacro:front_wheel_lr
@@ -98,11 +99,10 @@
         base_length="${base_length}"
         base_width="${base_width}"
-        axle_offset="${axle_offset}"
+        axle_length_offset="${axle_length_offset}"
+        axle_width_offset="${axle_width_offset}"
         steer_height="${wheel_radius+steer_offset}"
-        model_rotate="1.57">
-        <origin xyz="0 0 0" rpy="${-90 * deg_to_rad} 0 0" />
+        model_rotate="0">
     </xacro:front_wheel_lr>
-    <!--Rear
-    Wheels -->
+    <!--Rear Wheels -->
     <xacro:rear_wheel_lr
         name="rear_right"
@@ -112,9 +112,9 @@
         wheel_thickness="${wheel_thickness}"
         wheel_mass="${wheel_mass}"
-        model_rotate="-1.57"
+        model_rotate="${pi}"
         base_length="${base_length}"
         base_width="${base_width}"
-        axle_offset="${axle_offset}"
-        steer_height="${wheel_radius+steer_offset}">
+        axle_length_offset="${axle_length_offset}"
+        axle_width_offset="${axle_width_offset}">
     </xacro:rear_wheel_lr>
     <xacro:rear_wheel_lr
@@ -125,9 +125,9 @@
         wheel_thickness="${wheel_thickness}"
         wheel_mass="${wheel_mass}"
-        model_rotate="1.57"
+        model_rotate="0"
         base_length="${base_length}"
         base_width="${base_width}"
-        axle_offset="${axle_offset}"
-        steer_height="${wheel_radius+steer_offset}">
+        axle_length_offset="${axle_length_offset}"
+        axle_width_offset="${axle_width_offset}">
     </xacro:rear_wheel_lr>
     <xacro:door
@@ -135,33 +135,4 @@
         parent="base">
     </xacro:door>
-    <!-- Realsense Camera
-    <xacro:realsense_camera
-        name="front"
-        parent="base_link"
-        orientation="${90 * deg_to_rad}"
-        mirror = "1">
-        <origin xyz="0.39875 0 0.575" rpy="0 0 0" />
-    </xacro:realsense_camera>
-    <xacro:realsense_camera
-        name="rear"
-        parent="base_link"
-        orientation="${90 * deg_to_rad}"
-        mirror = "-1">
-        <origin xyz="-0.39875 0 0.575" rpy="0 0 ${180 * deg_to_rad}" />
-    </xacro:realsense_camera> -->
-    <!-- <xacro:depth_camera
-        name="front"
-        parent="base_link"
-        orientation="0"
-        mirror = "1">
-        <origin xyz="0.39875 0 0.575" rpy="0 0 0" />
-    </xacro:depth_camera>
-    <xacro:depth_camera
-        name="rear"
-        parent="base_link"
-        orientation="${-90 * deg_to_rad}"
-        mirror = "-1">
-        <origin xyz="-0.39875 0 0.575" rpy="0 0 ${180 * deg_to_rad}" />
-    </xacro:depth_camera> -->
     <ros2_control name="GazeboSystem" type="system">
         <hardware>

File: deliverybot_description/models/deliverybot/xacro/deliverybot_joints.xacro (robot description, xacro)
@@ -19,8 +19,8 @@
         base_length
         base_width
-        axle_offset
+        axle_length_offset
+        axle_width_offset
         steer_height
-        model_rotate
-        *origin">
+        model_rotate">
         <link name="${name}_steer_link">
             <inertial>
@@ -39,5 +39,5 @@
             <child link="${name}_steer_link" />
             <origin
-                xyz="${base_length/2-axle_offset} ${reflect*(base_width/2+axle_offset)} ${steer_height}"
+                xyz="${reflect*(base_width/2)} ${base_length/2-axle_length_offset} ${-0.345}"
                 rpy="0 0 0" />
             <axis xyz="0 0 1" />
@@ -49,5 +49,5 @@
         <link name="${name}_wheel_link">
             <visual>
-                <origin xyz="0 0 0" rpy="0 ${model_rotate} 1.57" />
+                <origin xyz="0 0 0" rpy="0 ${model_rotate} 0" />
                 <geometry>
                     <mesh
@@ -56,5 +56,5 @@
             </visual>
             <collision>
-                <origin xyz="0 0 0" rpy="0 ${model_rotate} 1.57" />
+                <origin xyz="0 0 0" rpy="0 ${model_rotate} 0" />
                 <geometry>
                     <mesh
@@ -71,5 +71,5 @@
             </collision>
             <inertial>
-                <origin xyz="0 0 0" rpy="0 ${model_rotate} 1.57" />
+                <origin xyz="0 0 0" rpy="0 0 0" />
                 <mass value="3.512" />
                 <inertia ixx="0.02665" ixy="0" ixz="0" iyy="0.0148" iyz="0" izz="0.01479" />
@@ -79,6 +79,6 @@
             <parent link="${name}_steer_link" />
             <child link="${name}_wheel_link" />
-            <xacro:insert_block name="origin" />
-            <axis xyz="0 0 1" />
+            <origin xyz="${reflect * (wheel_thickness)} 0 0" rpy="${-90 * deg_to_rad} ${-pi} 0" />
+            <axis xyz="1 0 0" />
         </joint>
         <gazebo reference="${name}_steer_link">
@@ -110,9 +110,9 @@
         base_length
         base_width
-        axle_offset
-        steer_height">
+        axle_length_offset
+        axle_width_offset">
         <link name="${name}_wheel_link">
             <visual>
-                <origin xyz="0 0 0" rpy="0 ${model_rotate} 1.57" />
+                <origin xyz="0 0 0" rpy="0 ${model_rotate} 0" />
                 <geometry>
                     <mesh
@@ -121,5 +121,5 @@
             </visual>
             <collision>
-                <origin xyz="0 0 0" rpy="0 ${model_rotate} 1.57" />
+                <origin xyz="0 0 0" rpy="0 ${model_rotate} 0" />
                 <geometry>
                     <mesh
@@ -136,5 +136,5 @@
             </collision>
             <inertial>
-                <origin xyz="0 0 0" rpy="0 0 0" />
+                <origin xyz="0 0 0" rpy="0 ${model_rotate} 0" />
                 <mass value="3.512" />
                 <inertia ixx="0.02665" ixy="0" ixz="0" iyy="0.0148" iyz="0" izz="0.01479" />
@@ -145,7 +145,7 @@
             <child link="${name}_wheel_link" />
             <origin
-                xyz="${-base_length/2+axle_offset} ${reflect*(base_width/2+axle_offset)} ${steer_height}"
-                rpy="${-90 * deg_to_rad} 0 0" />
-            <axis xyz="0 0 1" />
+                xyz="${reflect*(base_width/2 + wheel_thickness)} ${-(base_length/2-axle_length_offset)} ${-0.345}"
+                rpy="${-90 * deg_to_rad} ${-pi} 0" />
+            <axis xyz="1 0 0" />
         </joint>
         <gazebo reference="${name}_wheel_link">
@@ -167,8 +167,8 @@
                         filename="package://deliverybot_description/models/deliverybot/meshes/EVA_Lid.dae" />
                 </geometry>
-                <origin rpy="0 0 ${-90 * deg_to_rad}" xyz="0.42300 0 0" />
+                <origin rpy="0 0 0" xyz="-0.002550 0.400 0.01750" />
             </visual>
             <collision>
-                <origin rpy="0 0 ${-90 * deg_to_rad}" xyz="0.42300 0 0" />
+                <origin rpy="0 0 0" xyz="0 0.400 0.01750" />
                 <geometry>
                     <mesh
@@ -177,5 +177,5 @@
             </collision>
             <inertial>
-                <origin rpy="0 0 -1.57" xyz="0 0 0" />
+                <origin rpy="0 0 0" xyz="0 0 0" />
                 <mass value="8" />
                 <inertia ixx="0.4381" ixy="0" ixz="0" iyy="0.1637" iyz="0.005" izz="0.6" />
@@ -183,9 +183,9 @@
         </link>
         <joint name="${name}_joint" type="revolute">
-            <limit lower="-1.57" upper="0" effort="100" velocity="0.5" />
-            <origin rpy="0 0 0" xyz="-0.4365 0.0025 0.695" />
+            <limit lower="0" upper="1.5708" effort="100" velocity="0.5" />
+            <origin rpy="0 0 0" xyz="0 -0.415 0.35250" />
             <parent link="${parent}_link" />
             <child link="${name}_link" />
-            <axis xyz="0 1 0" rpy="0 0 0" />
+            <axis xyz="1 0 0" rpy="0 0 0" />
         </joint>
     </xacro:macro>

Commit message: Fixed MAP Frame visualization in RVIZ

File: deliverybot_description/models/deliverybot/xacro/deliverybot.xacro (robot description, xacro)
@@ -40,5 +40,4 @@
     <!-- Dummy Link -->
     <link name="base_footprint" />
-    <!-- <link name="map" /> -->
     <!-- Base Link -->
     <link name="base_link">

Commit message: Modified file structure and code cleanup

File: deliverybot_description/models/deliverybot/xacro/deliverybot.xacro (robot description, xacro)
@@ -46,5 +46,5 @@
             <geometry>
                 <mesh
-                    filename="package://deliverybot_description/models/deliverybot/meshes/EVA_Body_new.dae" />
+                    filename="package://deliverybot_description/models/deliverybot/meshes/EVA_Body.dae" />
             </geometry>
         </visual>
@@ -53,5 +53,5 @@
             <geometry>
                 <mesh
-                    filename="package://deliverybot_description/models/deliverybot/meshes/EVA_Body_new.dae" />
+                    filename="package://deliverybot_description/models/deliverybot/meshes/EVA_Body.dae" />
             </geometry>
         </collision>

File: deliverybot_description/models/deliverybot/xacro/slam.xacro (robot description, xacro)
@@ -9,5 +9,5 @@
         name="front"
         parent="base_link"
-        orientation="${180 * deg_to_rad}"
+        orientation="${90 * deg_to_rad}"
         mirror="-1">
         <origin xyz="0 0.39875 0.25250" rpy="0 0 ${90*deg_to_rad}" />
@@ -16,7 +16,7 @@
         name="rear"
         parent="base_link"
-        orientation="${180 * deg_to_rad}"
+        orientation="${-90 * deg_to_rad}"
         mirror="1">
-        <origin xyz="0 -0.39875 0.25250" rpy="0 0 ${90 * deg_to_rad}" />
+        <origin xyz="0 -0.39875 0.25250" rpy="0 0 ${-90 * deg_to_rad}" />
     </xacro:realsense_camera>
 </robot>

Commit message: Working wheel/imu odometry - starting slam

File: deliverybot_description/models/deliverybot/xacro/deliverybot.xacro (robot description, xacro)
@@ -35,5 +35,5 @@
     <!-- Axle Positions -->
     <xacro:property name="axle_length_offset" value="0.125" />
-    <xacro:property name="axle_width_offset" value="0.1"/>
+    <xacro:property name="axle_width_offset" value="0.1" />
     <xacro:property name="steer_offset" value="-0.15" />
     <!-- Dummy Link -->
@@ -63,7 +63,27 @@
     <!-- Dummy Joint -->
     <joint name="base_joint" type="fixed">
-        <origin xyz="0 0 0.470" rpy="0 0 0"/>
+        <origin xyz="0 0 0.470" rpy="0 0 0" />
         <parent link="base_footprint" />
         <child link="base_link" />
+    </joint>
+    <link name="center_steer_link">
+        <inertial>
+            <origin rpy="0 0 0" xyz="0 0 0" />
+            <mass value="${steer_mass}" />
+            <inertia
+                ixx="${steer_mass * (3.0 * steer_radius * steer_radius + steer_thickness * steer_thickness) / 12.0}"
+                ixy="0.0" ixz="0.0"
+                iyy="${steer_mass * (3.0 * steer_radius * steer_radius + steer_thickness * steer_thickness) / 12.0}"
+                iyz="0.0"
+                izz="${steer_mass * (steer_radius * steer_radius) / 2.0}" />
+        </inertial>
+    </link>
+    <joint name="center_steer_joint" type="revolute">
+        <parent link="base_link" />
+        <child link="center_steer_link" />
+        <origin xyz="0 ${base_length/2 - axle_length_offset} -0.345" rpy="0 0 0" />
+        <axis xyz="0 0 1" />
+        <limit effort="${steer_effort}" lower="${steer_limit_deg * deg_to_rad * -1.0}"
+            upper="${steer_limit_deg * deg_to_rad}" velocity="${steer_velocity}" />
     </joint>
     <!-- Steerable Front Wheels -->
@@ -102,5 +122,6 @@
         model_rotate="0">
     </xacro:front_wheel_lr>
-    <!--Rear Wheels -->
+    <!--Rear
+    Wheels -->
     <xacro:rear_wheel_lr
         name="rear_right"
@@ -145,4 +166,8 @@
             steer_limlow="${steer_limlow_deg * deg_to_rad}"
             steer_limhigh="${steer_limhigh_deg * deg_to_rad}" />
+        <xacro:steering_control
+            name="center"
+            steer_limlow="${steer_limlow_deg * deg_to_rad}"
+            steer_limhigh="${steer_limhigh_deg * deg_to_rad}" />
         <xacro:door_control
             name="door"

File: deliverybot_description/models/deliverybot/xacro/nav2.xacro (robot description, xacro)
@@ -4,7 +4,7 @@
         filename="$(find deliverybot_description)/models/deliverybot/xacro/deliverybot.xacro" />
     <xacro:include
-        filename="$(find deliverybot_description)/models/deliverybot/xacro/cameras.xacro" />
+        filename="$(find deliverybot_description)/models/deliverybot/xacro/sensors.xacro" />
     <!-- Realsense Camera -->
-    <xacro:realsense_camera
+    <!-- <xacro:realsense_camera
         name="front"
         parent="base_link"
@@ -12,6 +12,6 @@
         mirror="-1">
         <origin xyz="0 0.39875 0.25250" rpy="0 0 ${90*deg_to_rad}" />
-    </xacro:realsense_camera>
-    <xacro:realsense_camera
+    </xacro:realsense_camera> -->
+    <!-- <xacro:realsense_camera
         name="rear"
         parent="base_link"
@@ -19,4 +19,16 @@
         mirror="1">
         <origin xyz="0 -0.39875 0.25250" rpy="0 0 ${-90 * deg_to_rad}" />
-    </xacro:realsense_camera>
+    </xacro:realsense_camera> -->
+    <xacro:depth_camera
+        name="front"
+        parent="base_link"
+        orientation="${90 * deg_to_rad}"
+        mirror="-1">
+        <origin xyz="0 0.39875 0.25250" rpy="0 0 ${90*deg_to_rad}" />
+    </xacro:depth_camera>
+    <xacro:lidar
+        name="top"
+        parent="base_link" />
+    <xacro:imu name="imu" parent="base_link"/>
+    <xacro:ackermann_odometry parent="base_link" />
 </robot>
