Commit message: 2D-Nav Goal and NAV2 Params

File: deliverybot_description/models/deliverybot/xacro/deliverybot.xacro (robot description, xacro)
@@ -38,9 +38,11 @@
     <xacro:property name="steer_offset" value="-0.15" />
     <!-- Dummy Link -->
-    <link name="base_footprint" />
+    <link name="base_footprint">
+        <origin xyz="0 0 0" rpy="0 0 0" />
+    </link>
     <!-- Base Link -->
     <link name="base_link">
         <visual>
-            <origin xyz="0 0 0" rpy="0 0 0" />
+            <origin xyz="0 0 0" rpy="0 0 ${-pi/2}" />
             <geometry>
                 <mesh
@@ -49,5 +51,5 @@
         </visual>
         <collision>
-            <origin xyz="0 0 0" rpy="0 0 0" />
+            <origin xyz="0 0 0" rpy="0 0 ${-pi/2}" />
             <geometry>
                 <mesh
@@ -56,5 +58,5 @@
         </collision>
         <inertial>
-            <origin xyz="0 0 0" rpy="0 0 0" />
+            <origin xyz="0 0 0" rpy="0 0 ${-pi/2}" />
             <mass value="64.3" />
             <inertia ixx="8.303" ixy="0" ixz="0" iyy="5.468" iyz="0.075" izz="6.02" />
@@ -82,5 +84,5 @@
         <parent link="base_link" />
         <child link="center_steer_link" />
-        <origin xyz="0 ${base_length/2 - axle_length_offset} -0.345" rpy="0 0 0" />
+        <origin xyz="${base_length/2 - axle_length_offset} 0 -0.345" rpy="0 0 0" />
         <axis xyz="0 0 1" />
         <limit effort="${steer_effort}" lower="${steer_limit_deg * deg_to_rad * -1.0}"
@@ -102,6 +104,5 @@
         axle_length_offset="${axle_length_offset}"
         axle_width_offset="${axle_width_offset}"
-        steer_height="${wheel_radius+steer_offset}"
-        model_rotate="${pi}">
+        steer_height="${wheel_radius+steer_offset}">
     </xacro:front_wheel_lr>
     <xacro:front_wheel_lr
@@ -119,9 +120,6 @@
         axle_length_offset="${axle_length_offset}"
         axle_width_offset="${axle_width_offset}"
-        steer_height="${wheel_radius+steer_offset}"
-        model_rotate="0">
+        steer_height="${wheel_radius+steer_offset}">
     </xacro:front_wheel_lr>
-    <!--Rear
-    Wheels -->
     <xacro:rear_wheel_lr
         name="rear_right"
@@ -131,5 +129,4 @@
         wheel_thickness="${wheel_thickness}"
         wheel_mass="${wheel_mass}"
-        model_rotate="${pi}"
         base_length="${base_length}"
         base_width="${base_width}"
@@ -144,5 +141,4 @@
         wheel_thickness="${wheel_thickness}"
         wheel_mass="${wheel_mass}"
-        model_rotate="0"
         base_length="${base_length}"
         base_width="${base_width}"
@@ -159,21 +155,21 @@
         </hardware>
         <xacro:steering_control
+            name="center"
+            steer_limlow="${steer_limlow_deg * deg_to_rad}"
+            steer_limhigh="${steer_limhigh_deg * deg_to_rad}" />
+        <xacro:steering_control
             name="front_right"
             steer_limlow="${steer_limlow_deg * deg_to_rad}"
             steer_limhigh="${steer_limhigh_deg * deg_to_rad}" />
+        <xacro:velocity_control
+            name="front_right"
+            velocity_limlow="${velocity_limlow}"
+            velocity_limhigh="${velocity_limhigh}" />
         <xacro:steering_control
             name="front_left"
             steer_limlow="${steer_limlow_deg * deg_to_rad}"
             steer_limhigh="${steer_limhigh_deg * deg_to_rad}" />
-        <xacro:steering_control
-            name="center"
-            steer_limlow="${steer_limlow_deg * deg_to_rad}"
-            steer_limhigh="${steer_limhigh_deg * deg_to_rad}" />
-        <xacro:door_control
-            name="door"
-            door_limlow="${0 * deg_to_rad}"
-            door_limhigh="${90 * deg_to_rad}" />
         <xacro:velocity_control
-            name="rear_left"
+            name="front_left"
             velocity_limlow="${velocity_limlow}"
             velocity_limhigh="${velocity_limhigh}" />
@@ -183,11 +179,11 @@
             velocity_limhigh="${velocity_limhigh}" />
         <xacro:velocity_control
-            name="front_right"
+            name="rear_left"
             velocity_limlow="${velocity_limlow}"
             velocity_limhigh="${velocity_limhigh}" />
-        <xacro:velocity_control
-            name="front_left"
-            velocity_limlow="${velocity_limlow}"
-            velocity_limhigh="${velocity_limhigh}" />
+        <xacro:door_control
+            name="door"
+            door_limlow="${0 * deg_to_rad}"
+            door_limhigh="${90 * deg_to_rad}" />
     </ros2_control>
 </robot>

File: deliverybot_description/models/deliverybot/xacro/deliverybot_joints.xacro (robot description, xacro)
@@ -5,6 +5,5 @@
         value="0.5" />
     <xacro:property name="steer_limit_deg" value="35.0" />
-    <xacro:macro
-        name="front_wheel_lr"
+    <xacro:macro name="front_wheel_lr"
         params="
         name
@@ -21,6 +20,5 @@
         axle_length_offset
         axle_width_offset
-        steer_height
-        model_rotate">
+        steer_height">
         <link name="${name}_steer_link">
             <inertial>
@@ -39,5 +37,5 @@
             <child link="${name}_steer_link" />
             <origin
-                xyz="${reflect*(base_width/2)} ${base_length/2-axle_length_offset} ${-0.345}"
+                xyz="${base_length/2-axle_length_offset} ${reflect*(base_width/2)} ${-0.345}"
                 rpy="0 0 0" />
             <axis xyz="0 0 1" />
@@ -49,5 +47,5 @@
         <link name="${name}_wheel_link">
             <visual>
-                <origin xyz="0 0 0" rpy="0 ${model_rotate} 0" />
+                <origin xyz="0 0 0" rpy="0 0 ${reflect * -pi/2}" />
                 <geometry>
                     <mesh
@@ -56,5 +54,5 @@
             </visual>
             <collision>
-                <origin xyz="0 0 0" rpy="0 ${model_rotate} 0" />
+                <origin xyz="0 0 0" rpy="0 0 ${reflect * -pi/2}" />
                 <geometry>
                     <mesh
@@ -79,6 +77,6 @@
             <parent link="${name}_steer_link" />
             <child link="${name}_wheel_link" />
-            <origin xyz="${reflect * (wheel_thickness)} 0 0" rpy="${-90 * deg_to_rad} ${-pi} 0" />
-            <axis xyz="1 0 0" />
+            <origin xyz="0 ${reflect * (wheel_thickness)} 0" rpy="0 0 0" />
+            <axis xyz="0 1 0" />
         </joint>
         <gazebo reference="${name}_steer_link">
@@ -98,6 +96,5 @@
     </xacro:macro>
     <!-- Rear Wheel Links -->
-    <xacro:macro
-        name="rear_wheel_lr"
+    <xacro:macro name="rear_wheel_lr"
         params="
         name
@@ -107,5 +104,4 @@
         wheel_thickness
         wheel_mass
-        model_rotate
         base_length
         base_width
@@ -114,5 +110,5 @@
         <link name="${name}_wheel_link">
             <visual>
-                <origin xyz="0 0 0" rpy="0 ${model_rotate} 0" />
+                <origin xyz="0 0 0" rpy="0 0 ${reflect * -pi/2}" />
                 <geometry>
                     <mesh
@@ -121,5 +117,5 @@
             </visual>
             <collision>
-                <origin xyz="0 0 0" rpy="0 ${model_rotate} 0" />
+                <origin xyz="0 0 0" rpy="0 0 ${reflect * -pi/2}" />
                 <geometry>
                     <mesh
@@ -136,5 +132,5 @@
             </collision>
             <inertial>
-                <origin xyz="0 0 0" rpy="0 ${model_rotate} 0" />
+                <origin xyz="0 0 0" rpy="0 0 ${reflect * -pi/2}" />
                 <mass value="3.512" />
                 <inertia ixx="0.02665" ixy="0" ixz="0" iyy="0.0148" iyz="0" izz="0.01479" />
@@ -145,7 +141,7 @@
             <child link="${name}_wheel_link" />
             <origin
-                xyz="${reflect*(base_width/2 + wheel_thickness)} ${-(base_length/2-axle_length_offset)} ${-0.345}"
-                rpy="${-90 * deg_to_rad} ${-pi} 0" />
-            <axis xyz="1 0 0" />
+                xyz="${-(base_length/2-axle_length_offset)} ${reflect*(base_width/2 + wheel_thickness)} ${-0.345}"
+                rpy="0 0 0" />
+            <axis xyz="0 1 0" />
         </joint>
         <gazebo reference="${name}_wheel_link">
@@ -167,8 +163,8 @@
                         filename="package://deliverybot_description/models/deliverybot/meshes/EVA_Lid.dae" />
                 </geometry>
-                <origin rpy="0 0 0" xyz="-0.002550 0.400 0.01750" />
+                <origin rpy="0 0 ${-pi/2}" xyz="0.400 -0.002550 0.01750" />
             </visual>
             <collision>
-                <origin rpy="0 0 0" xyz="-0.002550 0.400 0.01750" />
+                <origin rpy="0 0 ${-pi/2}" xyz="0.400 -0.002550 0.01750" />
                 <geometry>
                     <mesh
@@ -184,8 +180,8 @@
         <joint name="${name}_joint" type="revolute">
             <limit lower="0" upper="1.5708" effort="100" velocity="0.5" />
-            <origin rpy="0 0 0" xyz="0 -0.415 0.35250" />
+            <origin rpy="0 0 0" xyz="-0.415 0 0.35250" />
             <parent link="${parent}_link" />
             <child link="${name}_link" />
-            <axis xyz="1 0 0" rpy="0 0 0" />
+            <axis xyz="0 1 0" rpy="0 0 0" />
         </joint>
     </xacro:macro>

File: deliverybot_description/models/deliverybot/xacro/nav2.xacro (robot description, xacro)
@@ -11,5 +11,5 @@
         orientation="${90 * deg_to_rad}"
         mirror="-1">
-        <origin xyz="0 0.39875 0.25250" rpy="0 0 ${90*deg_to_rad}" />
+        <origin xyz="0.39875 0 0.25250" rpy="0 0 0" />
     </xacro:realsense_camera>
     <xacro:realsense_camera
@@ -18,16 +18,11 @@
         orientation="${90 * deg_to_rad}"
         mirror="1">
-        <origin xyz="0 -0.39875 0.25250" rpy="0 0 ${-90 * deg_to_rad}" />
+        <origin xyz="-0.39875 0 0.25250" rpy="0 0 ${180 * deg_to_rad}" />
     </xacro:realsense_camera>
-    <!-- <xacro:depth_camera
-        name="front"
-        parent="base_link"
-        orientation="${90 * deg_to_rad}"
-        mirror="-1">
-        <origin xyz="0 0.39875 0.25250" rpy="0 0 ${90*deg_to_rad}" />
-    </xacro:depth_camera> -->
     <xacro:lidar
         name="top"
-        parent="base_link" />
+        parent="base_link">
+        <origin xyz="-0.355 0 0.510" rpy="0 0 0" />
+    </xacro:lidar>
     <xacro:imu name="imu" parent="base_link"/>
     <xacro:ackermann_odometry parent="base_link" />

File: deliverybot_description/models/deliverybot/xacro/sensors.xacro (robot description, xacro)
@@ -8,5 +8,4 @@
         mirror
         *origin">
-        <!-- Visual Component -->
         <link name="${name}_rgb_link_optical" />
         <joint name="${name}_rgb_joint_optical" type="fixed">
@@ -45,5 +44,4 @@
             </sensor>
         </gazebo>
-        <!-- Depth Component -->
         <link name="${name}_depth_link">
             <visual>
@@ -90,5 +88,5 @@
                     <image>
                         <width>424</width>
-                        <height>240</height>
+                        <height>120</height>
                         <format>B8G8R8</format>
                     </image>
@@ -119,5 +117,6 @@
         params="
         name
-        parent">
+        parent
+        *origin">
         <link name="${name}_lidar_link">
             <inertial>
@@ -148,10 +147,10 @@
             <parent link="${parent}" />
             <child link="${name}_lidar_link" />
-            <origin xyz="0 -0.355 0.510" rpy="0 0 0" />
+            <xacro:insert_block name="origin"/>
         </joint>
         <gazebo reference="${name}_lidar_link">
             <sensor name="velodyne" type="ray">
                 <always_on>true</always_on>
-                <visualize>true</visualize>
+                <visualize>false</visualize>
                 <pose>0.0 0 0.0 0 0 0</pose>
                 <update_rate>15</update_rate>
@@ -178,81 +177,8 @@
                 <plugin name="velodyne_laserscan" filename="libgazebo_ros_ray_sensor.so">
                     <ros>
-                        <!-- <namespace>lidar</namespace> -->
                         <remapping>~/out:=scan</remapping>
                     </ros>
                     <output_type>sensor_msgs/LaserScan</output_type>
                     <frame_name>${name}_lidar_link</frame_name>
-                </plugin>
-            </sensor>
-        </gazebo>
-    </xacro:macro>
-    <xacro:macro name="depth_camera" params="name parent orientation mirror *origin">
-        <link name="${name}_depth_link">
-            <visual>
-                <origin xyz="0 0 0" rpy="0 0 ${orientation}" />
-                <geometry>
-                    <mesh
-                        filename="package://deliverybot_description/models/deliverybot/meshes/IntelRealsense.dae"
-                        scale="0.1 0.1 0.1" />
-                </geometry>
-            </visual>
-            <collision>
-                <origin xyz="0 0 0" rpy="0 0 ${orientation}" />
-                <geometry>
-                    <mesh
-                        filename="package://deliverybot_description/models/deliverybot/meshes/IntelRealsense.dae"
-                        scale="0.1 0.1 0.1" />
-                </geometry>
-            </collision>
-            <inertial>
-                <origin xyz="0 0 0" rpy="0 0 ${orientation}" />
-                <mass value="0.1" />
-                <inertia ixx="0.001" ixy="0" ixz="0" iyy="0.005" iyz="0" izz="0.005" />
-            </inertial>
-        </link>
-        <link name="${name}_depth_link_optical" />
-        <joint name="${name}_depth_joint" type="fixed">
-            <parent link="${parent}" />
-            <child link="${name}_depth_link" />
-            <xacro:insert_block name="origin" />
-        </joint>
-        <joint name="${name}_depth_joint_optical" type="fixed">
-            <origin xyz="0 0 0" rpy="${-pi/2} 0 ${-pi/2}" />
-            <parent link="${name}_depth_link" />
-            <child link="${name}_depth_link_optical" />
-        </joint>
-        <gazebo reference="${name}_depth_link">
-            <sensor name="${name}_depth_camera" type="depth">
-                <visualize>true</visualize>
-                <update_rate>30.0</update_rate>
-                <camera name="${name}_camera">
-                    <horizontal_fov>1.487021</horizontal_fov>
-                    <image>
-                        <width>640</width>
-                        <height>480</height>
-                        <format>B8G8R8</format>
-                    </image>
-                    <clip>
-                        <near>0.05</near>
-                        <far>3</far>
-                    </clip>
-                </camera>
-                <plugin name="${name}_depth_camera_controller" filename="libgazebo_ros_camera.so">
-                    <baseline>0.2</baseline>
-                    <alwaysOn>true</alwaysOn>
-                    <updateRate>0.0</updateRate>
-                    <frame_name>${name}_depth_joint_optical</frame_name>
-                    <pointCloudCutoff>0.5</pointCloudCutoff>
-                    <pointCloudCutoffMax>3.0</pointCloudCutoffMax>
-                    <distortionK1>0</distortionK1>
-                    <distortionK2>0</distortionK2>
-                    <distortionK3>0</distortionK3>
-                    <distortionT1>0</distortionT1>
-                    <distortionT2>0</distortionT2>
-                    <CxPrime>0</CxPrime>
-                    <Cx>0</Cx>
-                    <Cy>0</Cy>
-                    <focalLength>0</focalLength>
-                    <hackBaseline>0</hackBaseline>
                 </plugin>
             </sensor>
@@ -264,5 +190,5 @@
             <parent link="${parent}" />
             <child link="${name}" />
-            <origin xyz="0 0 0.1" rpy="0 0 0" />
+            <origin xyz="0 0 0" rpy="0 0 0" />
         </joint>
         <gazebo reference="${name}">
@@ -270,7 +196,7 @@
                 <plugin filename="libgazebo_ros_imu_sensor.so" name="imu_plugin">
                     <ros>
-                        <!-- <namespace>/demo</namespace> -->
                         <remapping>~/out:=imu</remapping>
                     </ros>
+                    <rpyOffset>0 0 1.5708</rpyOffset>
                     <initial_orientation_as_reference>false</initial_orientation_as_reference>
                 </plugin>
@@ -343,5 +269,5 @@
                     <remapping>distance:=wheel/distance</remapping>
                 </ros>
-                <!-- Wheels -->
+                <initial_orientation_as_reference>true</initial_orientation_as_reference>
                 <front_left_joint>front_left_wheel_joint</front_left_joint>
                 <front_right_joint>front_right_wheel_joint</front_right_joint>
@@ -351,9 +277,7 @@
                 <right_steering_joint>front_right_steer_joint</right_steering_joint>
                 <steering_wheel_joint>center_steer_joint</steering_wheel_joint>
-                <!-- Max absolute steer angle for tyre in radians -->
+                <rpyOffset>0 0 1.5708</rpyOffset>
                 <max_steer>0.610865</max_steer>
-                <!-- Max absolute linear speed in m/s -->
                 <max_speed>15</max_speed>
-                <!-- PID Tuning -->
                 <left_steering_pid_gain>1500 0 1</left_steering_pid_gain>
                 <left_steering_i_range>0 0</left_steering_i_range>
@@ -362,9 +286,8 @@
                 <linear_velocity_pid_gain>1000 0 1</linear_velocity_pid_gain>
                 <linear_velocity_i_range>0 0</linear_velocity_i_range>
-                <!-- output -->
                 <publish_odom>true</publish_odom>
                 <publish_odom_tf>false</publish_odom_tf>
                 <publish_wheel_tf>false</publish_wheel_tf>
-                <publish_distance>true</publish_distance>
+                <publish_distance>false</publish_distance>
                 <odometry_frame>odom</odometry_frame>
                 <robot_base_frame>base_footprint</robot_base_frame>

Commit message: Door joint actuation limits corrected

File: deliverybot_description/models/deliverybot/xacro/deliverybot.xacro (robot description, xacro)
@@ -185,5 +185,5 @@
             name="door"
             door_limlow="${0 * deg_to_rad}"
-            door_limhigh="${90 * deg_to_rad}" />
+            door_limhigh="${-90 * deg_to_rad}" />
     </ros2_control>
 </robot>

File: deliverybot_description/models/deliverybot/xacro/deliverybot_joints.xacro (robot description, xacro)
@@ -179,5 +179,5 @@
         </link>
         <joint name="${name}_joint" type="revolute">
-            <limit lower="0" upper="1.5708" effort="100" velocity="0.5" />
+            <limit lower="0" upper="-1.5708" effort="100" velocity="0.5" />
             <origin rpy="0 0 0" xyz="-0.415 0 0.35250" />
             <parent link="${parent}_link" />

Commit message: Cleanup

File: deliverybot_description/models/deliverybot/xacro/deliverybot.xacro (robot description, xacro)
@@ -60,5 +60,5 @@
             <origin xyz="0 0 0" rpy="0 0 ${-pi/2}" />
             <mass value="64.3" />
-            <inertia ixx="8.303" ixy="0" ixz="0" iyy="5.468" iyz="0.075" izz="6.02" />
+            <inertia ixx="8.303" ixy="0" ixz="0" iyy="5.468" iyz="0.00" izz="6.02" />
         </inertial>
     </link>
